Commit message: Added keyboard input and propeller forces

File: boat_sim/imarc_description/urdf/imarc.xacro (robot description, xacro)
@@ -3,5 +3,5 @@
 <xacro:property name="namespace" value="imarc"/>
 <!-- mass in kg, volume in m^3 123.225, -->
-<xacro:property name="mass" value="12"/>
+<xacro:property name="mass" value="123.225"/>
 <xacro:property name="volume" value="0.274"/>
 <xacro:property name="length" value="1.219"/>
@@ -17,5 +17,5 @@
 			</geometry>
 		</visual>
-		<collision>
+		<collision >
 			<origin xyz="0 0 0" rpy="0 0 0"/>
 			<geometry>
@@ -27,4 +27,54 @@
 		<mass value="${mass}"/>
 		<inertia ixx="${(width*width + depth*depth)*mass/12.0 }"  ixy="0"  ixz="0" iyy="${(length*length + depth*depth)*mass/12.0}" iyz="0" izz="${(length*length + depth*depth)*mass/12.0}"/>
+		</inertial>
+	</link>
+	<joint name="prop_joint_l" type="fixed">
+	    <axis xyz="0 1 0" />
+	    <origin xyz="${-length*0.5} ${-width*0.33} 0" rpy="0 0 0"/>
+	    <parent link="body"/>
+	    <child link="prop_l"/>
+	</joint>
+	<joint name="prop_joint_r" type="fixed">
+	    <axis xyz="0 1 0" />
+	    <origin xyz="${-length*0.5} ${width*0.33} 0" rpy="0 0 0"/>
+	    <parent link="body"/>
+	    <child link="prop_r"/>
+	</joint>
+	<link name="prop_l">
+		<collision>
+		  <origin xyz="0 0 0" rpy="0 0 0"/>
+		  <geometry>
+		    <box size="0.1 0.1 0.1"/>
+		  </geometry>
+		</collision>
+		<visual>
+		  <origin xyz="0 0 0" rpy="0 0 0"/>
+		  <geometry>
+		    <box size="0.1 0.1 0.1"/>
+		  </geometry>
+		</visual>
+		<inertial>
+		  <mass value="1e-5" />
+		  <origin xyz="0 0 0" rpy="0 0 0"/>
+		  <inertia ixx="1e-6" ixy="0" ixz="0" iyy="1e-6" iyz="0" izz="1e-6"/>
+		</inertial>
+	</link>
+	<link name="prop_r">
+		<collision>
+		  <origin xyz="0 0 0" rpy="0 0 0"/>
+		  <geometry>
+		    <box size="0.1 0.1 0.1"/>
+		  </geometry>
+		</collision>
+		<visual>
+		  <origin xyz="0 0 0" rpy="0 0 0"/>
+		  <geometry>
+		    <box size="0.1 0.1 0.1"/>
+		  </geometry>
+		</visual>
+		<inertial>
+		  <mass value="1e-5" />
+		  <origin xyz="0 0 0" rpy="0 0 0"/>
+		  <inertia ixx="1e-6" ixy="0" ixz="0" iyy="1e-6" iyz="0" izz="1e-6"/>
 		</inertial>
 	</link>

Commit message: Props work, imu, camera added

File: boat_sim/imarc_description/urdf/imarc.xacro (robot description, xacro)
@@ -8,4 +8,5 @@
 <xacro:property name="width" value="0.737"/>
 <xacro:property name="depth" value="0.3048"/>
+<xacro:property name="camera_link" value="0.05" /> <!-- Size of square 'camera' box -->
 <xacro:include filename="$(find imarc_description)/urdf/imarc.gazebo"/>
 <!-- TODO: maybe calc center of buoyancy -->
@@ -105,3 +106,30 @@
 		</inertial>
 	</link>
+  <joint name="camera_joint" type="fixed">
+    <axis xyz="0 1 0" />
+	<origin xyz="${length*0.4} ${-width*0.33} ${depth*0.5}" rpy="0 0 0"/>
+    <parent link="body"/>
+    <child link="camera_link"/>
+  </joint>
+  <!-- Camera -->
+  <link name="camera_link">
+    <collision>
+      <origin xyz="0 0 0" rpy="0 0 0"/>
+      <geometry>
+		<box size="${camera_link} ${camera_link} ${camera_link}"/>
+      </geometry>
+    </collision>
+    <visual>
+      <origin xyz="0 0 0" rpy="0 0 0"/>
+      <geometry>
+    <box size="${camera_link} ${camera_link} ${camera_link}"/>
+      </geometry>
+      <material name="red"/>
+    </visual>
+    <inertial>
+      <mass value="1e-5" />
+      <origin xyz="0 0 0" rpy="0 0 0"/>
+      <inertia ixx="1e-6" ixy="0" ixz="0" iyy="1e-6" iyz="0" izz="1e-6" />
+    </inertial>
+  </link>
 </robot>

Commit message: Working tf publishing, Rpi pwm generation, dutycycle publishing

File: boat_sim/imarc_description/urdf/imarc.xacro (robot description, xacro)
@@ -5,4 +5,5 @@
 <xacro:property name="mass" value="123.225"/>
 <xacro:property name="volume" value="0.274"/>
+<xacro:property name="pi" value="3.1415926535897931"/>
 <xacro:property name="length" value="1.219"/>
 <xacro:property name="width" value="0.737"/>
@@ -18,5 +19,5 @@
 			</geometry>
 		</visual>
-		<collision >
+		<collision name="body_collision">
 			<origin xyz="0 0 0" rpy="0 0 0"/>
 			<geometry>
@@ -30,4 +31,5 @@
 		</inertial>
 	</link>
+<!--
 	<joint name="prop_joint_l" type="fixed">
 	    <axis xyz="0 1 0" />
@@ -43,5 +45,5 @@
 	</joint>
 	<link name="prop_l">
-		<collision>
+		<collision name="prop_l_collision">
 		  <origin xyz="0 0 0" rpy="0 0 0"/>
 		  <geometry>
@@ -62,5 +64,5 @@
 	</link>
 	<link name="prop_r">
-		<collision>
+		<collision name="prop_r_collision">
 		  <origin xyz="0 0 0" rpy="0 0 0"/>
 		  <geometry>
@@ -80,4 +82,5 @@
 		</inertial>
 	</link>
+-->
   <joint name="hokuyo_joint" type="fixed">
     <axis xyz="0 1 0" />
@@ -88,5 +91,5 @@
 	<!-- Hokuyo Laser -->
 	<link name="hokuyo_link">
-		<collision>
+		<collision name="laser_collision">
 		  <origin xyz="0 0 0" rpy="0 0 0"/>
 		  <geometry>
@@ -114,5 +117,5 @@
   <!-- Camera -->
   <link name="camera_link">
-    <collision>
+    <collision name="camera_collision">
       <origin xyz="0 0 0" rpy="0 0 0"/>
       <geometry>
@@ -133,3 +136,14 @@
     </inertial>
   </link>
+  <!-- generate an optical frame http://www.ros.org/reps/rep-0103.html#suffix-frames
+      so that ros and opencv can operate on the camera frame correctly -->
+  <joint name="camera_optical_joint" type="fixed">
+    <!-- these values have to be these values otherwise the gazebo camera image
+        won't be aligned properly with the frame it is supposedly originating from -->
+    <origin xyz="0 0 0" rpy="${-pi/2} 0 ${-pi/2}"/>
+    <parent link="camera_link"/>
+    <child link="camera_link_optical"/>
+  </joint>
+  <link name="camera_link_optical">
+  </link>
 </robot>

Commit message: lidar test

File: boat_sim/imarc_description/urdf/imarc.xacro (robot description, xacro)
@@ -87,26 +87,26 @@
     <origin xyz="0 0 ${depth*0.5}" rpy="0 0 0"/>
     <parent link="body"/>
-    <child link="hokuyo_link"/>
+    <child link="laser_frame"/>
   </joint>
-	<!-- Hokuyo Laser -->
-	<link name="hokuyo_link">
-		<collision name="laser_collision">
-		  <origin xyz="0 0 0" rpy="0 0 0"/>
-		  <geometry>
-		    <box size="0.1 0.1 0.1"/>
-		  </geometry>
-		</collision>
-		<visual>
-		  <origin xyz="0 0 0" rpy="0 0 0"/>
-		  <geometry>
-		    <box size="0.1 0.1 0.1"/>
-		  </geometry>
-		</visual>
-		<inertial>
-		  <mass value="1e-5" />
-		  <origin xyz="0 0 0" rpy="0 0 0"/>
-		  <inertia ixx="1e-6" ixy="0" ixz="0" iyy="1e-6" iyz="0" izz="1e-6"/>
-		</inertial>
-	</link>
+<!-- Hokuyo Laser -->
+<link name="laser_frame">
+	<collision>
+	  <origin xyz="0 0 0" rpy="0 0 0"/>
+	  <geometry>
+	    <box size="0.1 0.1 0.1"/>
+	  </geometry>
+	</collision>
+	<visual>
+	  <origin xyz="0 0 0" rpy="0 0 0"/>
+	  <geometry>
+	    <box size="0.1 0.1 0.1"/>
+	  </geometry>
+	</visual>
+	<inertial>
+	  <mass value="1e-5" />
+	  <origin xyz="0 0 0" rpy="0 0 0"/>
+	  <inertia ixx="1e-6" ixy="0" ixz="0" iyy="1e-6" iyz="0" izz="1e-6"/>
+	</inertial>
+</link>
   <joint name="camera_joint" type="fixed">
     <axis xyz="0 1 0" />
